Commit message: change for me

File: src/week8_gazebo/urdf/rc_car.urdf (robot description, URDF)
Before this commit: robot rc_car, 5 links, 3 joints
Links:
- removed link rear_caster
- added link base_footprint
- added link camera_link; collision box size=0.0028125 0.005625 0.0050625
- added link camera_rgb_frame
- added link camera_rgb_optical_frame
- added link rear_left_wheel, mass 2.8125; collision cylinder length=0.028125 radius=0.028125; visual cylinder length=0.028125 radius=0.028125
- added link rear_right_wheel, mass 2.8125; collision cylinder length=0.028125 radius=0.028125; visual cylinder length=0.028125 radius=0.028125
- link base_link: mass 1.0 -> 168.75; geometry collision box size=0.225 0.1125 0.075; visual box size=0.225 0.1125 0.075
- link front_left_wheel: mass 0.1 -> 2.8125; geometry collision cylinder length=0.028125 radius=0.028125; visual cylinder length=0.028125 radius=0.028125
- link front_right_wheel: mass 0.1 -> 2.8125; geometry collision cylinder length=0.028125 radius=0.028125; visual cylinder length=0.028125 radius=0.028125
- link imu_link: mass 0.05 -> 0.1875; geometry visual box size=0.009375 0.009375 0.009375
Joints:
- removed joint rear_caster_joint
- added joint base_joint: type fixed, parent base_footprint, child base_link, origin xyz=0 0 0 rpy=0 0 0
- added joint camera_joint: type fixed, parent base_link, child camera_link, origin xyz=0.0136875 -0.0020625 0.01575 rpy=0 0 0
- added joint camera_rgb_joint: type fixed, parent camera_link, child camera_rgb_frame, origin xyz=0.0005625 0.0020625 0.0016875 rpy=0 0 0
- added joint camera_rgb_optical_joint: type fixed, parent camera_rgb_frame, child camera_rgb_optical_frame, origin xyz=0 0 0 rpy=-1.57 0 -1.57
- added joint imu_joint: type fixed, parent base_link, child imu_link, origin xyz=0 0 0.05625 rpy=0 0 0
- added joint rear_left_wheel_joint: type continuous, parent base_link, child rear_left_wheel, origin xyz=-0.1125 0.05625 0 rpy=0 0 0, axis 0 1 0
- added joint rear_right_wheel_joint: type continuous, parent base_link, child rear_right_wheel, origin xyz=-0.1125 -0.05625 0 rpy=0 0 0, axis 0 1 0
- joint front_left_wheel_joint: origin xyz=0.1 0.07 0.03 rpy=0 0 0 -> xyz=0.1125 0.05625 0 rpy=0 0 0
- joint front_right_wheel_joint: origin xyz=0.1 -0.07 0.03 rpy=0 0 0 -> xyz=0.1125 -0.05625 0 rpy=0 0 0

File: src/week8_gazebo/urdf/turtlebot3_waffle.urdf (robot description, URDF)
Before this commit: robot turtlebot3_burger, 10 links, 9 joints
Links:
- removed link caster_back_link
- added link camera_depth_frame
- added link camera_depth_optical_frame
- added link caster_back_left_link, mass 0.005; collision box size=0.030 0.009 0.020
- added link caster_back_right_link, mass 0.005; collision box size=0.030 0.009 0.020
- link base_link: mass 8.2573504e-01 -> 1.3729096e+00; geometry collision box size=0.266 0.266 0.094; visual mesh filename=package://turtlebot3_gazebo/models/turtlebot3_common/meshes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 scale=0.001 0.001 0.001
- link camera_link: geometry collision box size=0.012 0.132 0.020; visual mesh filename=package://turtlebot3_gazebo/models/turtlebot3_common/meshes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
Joints:
- removed joint caster_back_joint
- added joint camera_depth_joint: type fixed, parent camera_link, child camera_depth_frame, origin xyz=0.005 0.028 0.013 rpy=0 0 0
- added joint camera_depth_optical_joint: type fixed, parent camera_depth_frame, child camera_depth_optical_frame, origin xyz=0 0 0 rpy=-1.57 0 -1.57
- added joint caster_back_left_joint: type fixed, parent base_link, child caster_back_left_link, origin xyz=-0.177 0.064 -0.004 rpy=-1.57 0 0
- added joint caster_back_right_joint: type fixed, parent base_link, child caster_back_right_link, origin xyz=-0.177 -0.064 -0.004 rpy=-1.57 0 0
- joint base_joint: origin xyz=0.0 0.0 0.010 rpy=0 0 0 -> xyz=0 0 0.010 rpy=0 0 0
- joint camera_joint: origin xyz=0.073 -0.011 0.084 rpy=0 0 0 -> xyz=0.064 -0.065 0.094 rpy=0 0 0
- joint camera_rgb_joint: origin xyz=0.003 0.011 0.009 rpy=0 0 0 -> xyz=0.005 0.018 0.013 rpy=0 0 0
- joint imu_joint: origin xyz=-0.032 0 0.068 rpy=0 0 0 -> xyz=0.0 0 0.068 rpy=0 0 0
- joint scan_joint: origin xyz=-0.032 0 0.172 rpy=0 0 0 -> xyz=-0.064 0 0.122 rpy=0 0 0
- joint wheel_left_joint: origin xyz=0.0 0.08 0.023 rpy=-1.57 0 0 -> xyz=0.0 0.144 0.023 rpy=-1.57 0 0
- joint wheel_right_joint: origin xyz=0.0 -0.080 0.023 rpy=-1.57 0 0 -> xyz=0.0 -0.144 0.023 rpy=-1.57 0 0

Commit message: ggg

File: src/week8_gazebo/urdf/rc_car.urdf (robot description, URDF)
Before this commit: robot red_car, 10 links, 9 joints
Links:
- removed link camera_link
- removed link camera_rgb_frame
- removed link camera_rgb_optical_frame
- removed link front_left_wheel
- removed link front_right_wheel
- added link wheel_left_link, mass 2.8125; collision cylinder length=0.02 radius=0.03; visual cylinder length=0.02 radius=0.03
- added link wheel_right_link, mass 2.8125; collision cylinder length=0.02 radius=0.03; visual cylinder length=0.02 radius=0.03
- link base_link: geometry collision box size=0.25 0.15 0.10; visual box size=0.25 0.15 0.10
- link imu_link: geometry visual box size=0.01 0.01 0.01
- link rear_left_wheel: geometry collision cylinder length=0.02 radius=0.03; visual cylinder length=0.02 radius=0.03
- link rear_right_wheel: geometry collision cylinder length=0.02 radius=0.03; visual cylinder length=0.02 radius=0.03
Joints:
- removed joint camera_joint
- removed joint camera_rgb_joint
- removed joint camera_rgb_optical_joint
- removed joint front_left_wheel_joint
- removed joint front_right_wheel_joint
- added joint wheel_left_joint: type continuous, parent base_link, child wheel_left_link, origin xyz=0.1 0.075 0.03 rpy=-1.57 0 0, axis 0 0 1
- added joint wheel_right_joint: type continuous, parent base_link, child wheel_right_link, origin xyz=0.1 -0.075 0.03 rpy=-1.57 0 0, axis 0 0 1
- joint base_joint: origin xyz=0 0 0 rpy=0 0 0 -> xyz=0 0 0.01 rpy=0 0 0
- joint imu_joint: origin xyz=0 0 0.05625 rpy=0 0 0 -> xyz=0 0 0.07 rpy=0 0 0
- joint rear_left_wheel_joint: axis 0 1 0 -> 0 0 1; origin xyz=-0.1125 0.05625 0 rpy=0 0 0 -> xyz=-0.1 0.075 0.03 rpy=-1.57 0 0
- joint rear_right_wheel_joint: axis 0 1 0 -> 0 0 1; origin xyz=-0.1125 -0.05625 0 rpy=0 0 0 -> xyz=-0.1 -0.075 0.03 rpy=-1.57 0 0
